File: hardware/schematic/schematic.kicad_sch (KiCad schematic)
At the start: 14 parts

Commit message: First working prototype
Parts:
- removed 1.5V-BT? (x4): Battery, symbol Device:Battery
- removed M?: Motor_Servo, symbol Motor:Motor_Servo
Connections:
- net at A-UNO.10 (A1): no longer LEFT-USS.3 (ECHO)
- net at A-UNO.7 (GND), LEFT-USS.4 (GND), RIGHT-USS.4 (GND)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: now also A-UNO.17 (D2); no longer A-UNO.15 (D0/RX)
- net at A-UNO.16 (D1/TX): no longer RIGHT-USS.2 (TRIG)
- net at A-UNO.18 (D3): now also RIGHT-USS.3 (ECHO)
- net at A-UNO.19 (D4): now also LEFT-USS.3 (ECHO); no longer LEFT-USS.2 (TRIG)
- net at A-UNO.23 (D8): now also DC-DRIVER.7 (IN2)
- net at A-UNO.24 (D9): now also DC-DRIVER.5 (IN1)
- net at A-UNO.27 (D12): now also RIGHT-USS.2 (TRIG)
- net at A-UNO.28 (D13): now also LEFT-USS.2 (TRIG)
- net at A-UNO.9 (A0): no longer RIGHT-USS.3 (ECHO)
- new net: A-UNO.25 (D10), DC-DRIVER.12 (IN4)
- new net: A-UNO.26 (D11), DC-DRIVER.10 (IN3)
